File: schematics/68012to68000.sch (KiCad schematic (older format))
At the start: 0 parts

Commit message: Add schematics for the adapter.
Parts:
- added J1: 68000, symbol 68000
- added U1: 68012RC, symbol 68012RC
Connections:
- new net +5V: J1.14 (VCC), J1.49 (VCC), U1.D2 (VCC), U1.E9 (VCC)
- new net AS: J1.6 (AS), U1.A2 (AS)
- new net BERR: J1.22 (BERR), U1.J1 (BERR)
- new net BG: J1.11 (BG), U1.C2 (BG)
- new net BGACK: J1.12 (BGACK), U1.C1 (BGACK)
- new net BR: J1.13 (BR), U1.D1 (BR)
- new net CLK: J1.15 (CLK), U1.E1 (CLK)
- new net DTACK: J1.10 (DTACK), U1.B1 (DTACK)
- new net E: J1.20 (E), U1.H1 (E)
- new net FC0: J1.28 (FC0), U1.K3 (FC0)
- new net FC1: J1.27 (FC1), U1.J3 (FC1)
- new net FC2: J1.26 (FC2), U1.K2 (FC2)
- new net GND: J1.16 (GND), J1.53 (GND), U1.D8 (GND), U1.D9 (GND), U1.E2 (GND), U1.E3 (GND)
- new net HALT: J1.17 (HALT), U1.F1 (HALT)
- new net IPL0: J1.25 (IPL0), U1.J2 (IPL0)
- new net IPL1: J1.24 (IPL1), U1.H3 (IPL1)
- new net IPL2: J1.23 (IPL2), U1.H2 (IPL2)
- new net LDS: J1.8 (LDS), U1.B2 (LDS)
- new net RESET: J1.18 (RESET), U1.F2 (RESET)
- new net RW: J1.9 (R/W), U1.C3 (R/W)
- new net UDS: J1.7 (UDS), U1.B3 (UDS)
- new net VMA: J1.19 (VMA), U1.G1 (VMA)
- new net VPA: J1.21 (VPA), U1.G2 (VPA)
Other:
- note added: "SOCKET"
