File: schematics/68012to68000.sch (KiCad schematic (older format))
At the start: 2 parts, among them J1 68000, U1 68012RC

Commit message: Generate netlist, start PCB design.
Parts:
- J1: footprint (none) -> Housings_DIP:DIP-64_W22.86mm
- U1: footprint (none) -> Sockets:PGA84
Connections:
- net D4: now reaches J1.1 (D4)
- net D4: now also U1.A5 (D4)
- net D3: now reaches J1.2 (D3)
- net D3: now also U1.B5 (D3)
- net A1: now reaches J1.29 (A1)
- net A1: now also U1.K4 (A1)
- net D2: now reaches J1.3 (D2)
- net D2: now also U1.A4 (D2)
- net A2: now reaches J1.30 (A2)
- net A2: now also U1.J5 (A2)
- net A3: now reaches J1.31 (A3)
- net A3: now also U1.K5 (A3)
- net A4: now reaches J1.32 (A4)
- net A4: now also U1.K6 (A4)
- net A5: now reaches J1.33 (A5)
- net A5: now also U1.J6 (A5)
- net A6: now reaches J1.34 (A6)
- net A6: now also U1.K7 (A6)
- net A7: now reaches J1.35 (A7)
- net A7: now also U1.K8 (A7)
- net A8: now reaches J1.36 (A8)
- net A8: now also U1.J7 (A8)
- net A9: now reaches J1.37 (A9)
- net A9: now also U1.K9 (A9)
- net A10: now reaches J1.38 (A10)
- net A10: now also U1.J8 (A10)
- net A11: now reaches J1.39 (A11)
- net A11: now also U1.J9 (A11)
- net D1: now reaches J1.4 (D1)
- net D1: now also U1.A3 (D1)
- net A12: now reaches J1.40 (A12)
- net A12: now also U1.H9 (A12)
- net A13: now reaches J1.41 (A13)
- net A13: now also U1.H8 (A13)
- net A14: now reaches J1.42 (A14)
- net A14: now also U1.J10 (A14)
- net A15: now reaches J1.43 (A15)
- net A15: now also U1.G9 (A15)
- net A16: now reaches J1.44 (A16)
- net A16: now also U1.H10 (A16)
- net A17: now reaches J1.45 (A17)
- net A17: now also U1.G10 (A17)
- net A18: now reaches J1.46 (A18)
- net A18: now also U1.F9 (A18)
- net A19: now reaches J1.47 (A19)
- net A19: now also U1.F10 (A19)
- net A20: now reaches J1.48 (A20)
- net A20: now also U1.E10 (A20)
- net D0: now reaches J1.5 (D0)
- net D0: now also U1.B4 (D0)
- net A21: now reaches J1.50 (A21)
- net A21: now also U1.D10 (A21)
- net A22: now reaches J1.51 (A22)
- net A22: now also U1.C10 (A22)
- net A23: now reaches J1.52 (A23)
- net A23: now also U1.C9 (A23)
- net D15: now reaches J1.54 (D15)
- net D15: now also U1.B10 (D15)
- net D14: now reaches J1.55 (D14)
- net D14: now also U1.B9 (D14)
- net D13: now reaches J1.56 (D13)
- net D13: now also U1.C8 (D13)
- net D12: now reaches J1.57 (D12)
- net D12: now also U1.A10 (D12)
- net D11: now reaches J1.58 (D11)
- net D11: now also U1.B8 (D11)
- net D10: now reaches J1.59 (D10)
- net D10: now also U1.A9 (D10)
- net D9: now reaches J1.60 (D9)
- net D9: now also U1.B7 (D9)
- net D8: now reaches J1.61 (D8)
- net D8: now also U1.A8 (D8)
- net D7: now reaches J1.62 (D7)
- net D7: now also U1.A7 (D7)
- net D6: now reaches J1.63 (D6)
- net D6: now also U1.B6 (D6)
- net D5: now reaches J1.64 (D5)
- net D5: now also U1.A6 (D5)
- no-connect marks 0 -> 8
